File: accel.kicad_sch (KiCad schematic)
At the start: 3 parts, among them U1 CH376T, U2 MPU-6050

Commit message: updates
Connections:
- net at A1.7 (D4): now also U1.13 (~{SCS})
Changed lines of the file:
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@@
+    (stroke (width 0) (type default) (color 0 0 0 0))
+  )
+  (wire (pts (xy 104.14 101.6) (xy 104.14 113.03))
     (stroke (width 0) (type default) (color 0 0 0 0))
   )
@@
     (stroke (width 0) (type default) (color 0 0 0 0))
   )
+  (wire (pts (xy 96.52 113.03) (xy 104.14 113.03))
+    (stroke (width 0) (type default) (color 0 0 0 0))
+  )
   (wire (pts (xy 135.89 121.92) (xy 144.78 121.92))
     (stroke (width 0) (type default) (color 0 0 0 0))
@@
     (stroke (width 0) (type default) (color 0 0 0 0))
   )
+  (wire (pts (xy 104.14 101.6) (xy 110.49 101.6))
+    (stroke (width 0) (type default) (color 0 0 0 0))
+  )
